Commit message: Added alternative control for all joints, camera and adaptations for noetic sensors. Also added 4 ss lidars for good coverage

File: rbcar_description/robots/versions/rbcar_roborder.urdf.xacro (robot description, xacro)
@@ -48,11 +48,8 @@
                     lr_reflect="-1" fr_reflect="-1" parent="base_link" />
 	<!-- SENSORS -->
-  <xacro:sensor_benewake_ce30d prefix="front_3d_lidar" parent="base_link" gpu="true">
-      <origin xyz="2.155 0.0 0.236" rpy="0 0 0"/>
-  </xacro:sensor_benewake_ce30d>
-  <xacro:sensor_rubedos_viper prefix="viper" parent="base_link">
-      <origin xyz="1.289 0.0 1.354" rpy="0 0.0 0.0"/>
-  </xacro:sensor_rubedos_viper>
-	<xacro:sensor_imu_hector prefix="imu" parent="base_link">
+  <xacro:elevator parent="base_link">
+		<origin xyz="0.0 0.0 0.6" rpy="0 0 0"/>
+	</xacro:elevator>
+  <xacro:sensor_imu_hector prefix="imu" parent="base_link">
 		<origin xyz="0.0 0.0 0.170" rpy="0 0 0"/>
 	</xacro:sensor_imu_hector>
@@ -60,10 +57,23 @@
 		<origin xyz="0.0 0 1.5" rpy="0 0 0"/>
 	</xacro:sensor_gps>
-  <xacro:elevator parent="base_link">
-		<origin xyz="0.0 0.0 0.6" rpy="0 0 0"/>
-	</xacro:elevator>
+  <xacro:sensor_benewake_ce30d prefix="front_ss_lidar" parent="base_link" prefix_topic='front_ss_lidar' gpu="false">
+      <origin xyz="2.155 0.0 0.236" rpy="0 0 0"/>
+  </xacro:sensor_benewake_ce30d>
+  <xacro:sensor_benewake_ce30d prefix="back_ss_lidar" parent="base_link" prefix_topic='back_ss_lidar' gpu="false">
+      <origin xyz="-0.1 0.0 0.236" rpy="0 0 3.14"/>
+  </xacro:sensor_benewake_ce30d>
+  <xacro:sensor_benewake_ce30d prefix="left_ss_lidar" parent="base_link" prefix_topic='left_ss_lidar' gpu="false">
+      <origin xyz="1.0 -0.8 0.236" rpy="0 0 -1.52"/>
+  </xacro:sensor_benewake_ce30d>
+  <xacro:sensor_benewake_ce30d prefix="right_ss_lidar" parent="base_link" prefix_topic='right_ss_lidar' gpu="false">
+      <origin xyz="1.0 0.8 0.236" rpy="0 0 1.52"/>
+  </xacro:sensor_benewake_ce30d>
   <xacro:sensor_axis_q8641 prefix="front_ptz_camera" parent="elevator_link" far="300" near="0.08">
     <origin xyz="0 0 0" rpy="0 0 0"/>
   </xacro:sensor_axis_q8641>
+  <!-- Adding Sensors for navigation - and autonomous driving . Custom vvalues due to instability of version 16-->
+  <!-- <xacro:sensor_rslidar prefix="rslidar" parent="elevator_link" prefix_topic="rslidar" range_min="0.2" range_max="150.0" hfov="360.0" hres="0.1" vfov="30.0" vres="0.2" fps="2.0" gpu="true">
+    <origin xyz="0 0 0" rpy="0 0 0"/>
+  </xacro:sensor_rslidar> -->
 <gazebo>
 <plugin name="ground_truth_controller" filename="librobotnik_gazebo_ground_truth_odom.so">

File: rbcar_description/urdf/bases/rbcar_base.gazebo.xacro (robot description, xacro)
@@ -2,12 +2,13 @@
 <robot xmlns:xacro="http://wiki.ros.org/xacro">
   <!-- ros control plugin -->
-  <xacro:macro name="ros_control">
-    <gazebo>
-      <plugin name="ros_control" filename="libgazebo_ros_control.so">
-        <controlPeriod>0.001</controlPeriod>
-	    <robotSimType>gazebo_ros_control/DefaultRobotHWSim</robotSimType>
-	    <legacyModeNS>false</legacyModeNS>
-      </plugin>
-    </gazebo>
+	<xacro:macro name="ros_control">
+		<gazebo>
+			<plugin name="ros_control" filename="libgazebo_ros_control.so">
+			<controlPeriod>0.001</controlPeriod>
+			<robotNamespace>/rbcar</robotNamespace>
+			<robotSimType>gazebo_ros_control/DefaultRobotHWSim</robotSimType>
+			<legacyModeNS>false</legacyModeNS>
+			</plugin>
+		</gazebo>
 	</xacro:macro>
   <!-- No Ackermann steering plugin -->
@@ -23,5 +24,5 @@
 	    </plugin>
 	  </gazebo>
-  </xacro:macro>
+</xacro:macro>
   <gazebo reference="base_footprint">
     <material>Gazebo/Green</material>

File: rbcar_description/urdf/structures/elevator.urdf.xacro (robot description, xacro)
@@ -37,5 +37,5 @@
       <child link="${prefix}elevator_link"/>
       <axis xyz="0 0 1"/>
-      <limit lower="0.0" upper="${spread}" effort="100.0" velocity="0.07"/>
+      <limit lower="0.0" upper="${spread}" effort="1000.0" velocity="0.07"/>
       <!--<xacro:insert_block name="origin" />-->
     </joint>
@@ -56,9 +56,11 @@
       <type>transmission_interface/SimpleTransmission</type>
       <joint name="${prefix}elevator_joint">
-        <hardwareInterface>hardware_interface/PositionJointInterface</hardwareInterface>
+        <hardwareInterface>hardware_interface/EffortJointInterface</hardwareInterface>
+        <!-- <hardwareInterface>hardware_interface/PositionJointInterface</hardwareInterface> -->
       </joint>
       <actuator name="${prefix}elevator_motor">
         <mechanicalReduction>1</mechanicalReduction>
-        <hardwareInterface>hardware_interface/PositionJointInterface</hardwareInterface>
+        <hardwareInterface>hardware_interface/EffortJointInterface</hardwareInterface>
+        <!-- <hardwareInterface>hardware_interface/PositionJointInterface</hardwareInterface> -->
       </actuator>
     </transmission>

File: rbcar_description/urdf/wheels/suspension_wheel_v3.urdf.xacro (robot description, xacro)
@@ -105,5 +105,5 @@
   </xacro:macro>
   <!-- The "wheel" macro defines an axle carrier, axle, and wheel. -->
-  <xacro:macro name="wheel" params="lr_prefix fr_prefix lr_reflect">
+  <xacro:macro name="wheel" params="lr_prefix fr_prefix lr_reflect ackerman_debug:=0">
     <link name="${lr_prefix}_${fr_prefix}_axle_carrier">
 	  <!-- visual>
@@ -134,6 +134,6 @@
       <type>transmission_interface/SimpleTransmission</type>
       <joint name="${lr_prefix}_${fr_prefix}_axle">
-        <!-- hardwareInterface>hardware_interface/EffortJointInterface</hardwareInterface -->
-        <hardwareInterface>hardware_interface/VelocityJointInterface</hardwareInterface>
+        <hardwareInterface>hardware_interface/EffortJointInterface</hardwareInterface>
+        <!-- <hardwareInterface>hardware_interface/VelocityJointInterface</hardwareInterface> -->
       </joint>
       <actuator name="${lr_prefix}_${fr_prefix}_axle_act">
@@ -177,4 +177,20 @@
       <material>Gazebo/Black</material>
     </gazebo>
+    <!-- Visualization Ackerman -->
+    <xacro:if value="${ackerman_debug == 1}"> <!-- this applies if we are setting the left wheel -->
+      <link name="${lr_prefix}_${fr_prefix}_wheel_axis">
+        <visual>
+          <origin xyz="0 0 0" rpy = "0 0 0"/>
+          <geometry>
+            <cylinder radius="0.05" length="10.0"/>
+          </geometry>
+          <material name="tire_mat"/>
+        </visual>
+      </link>
+      <joint name="${lr_prefix}_${fr_prefix}_ackerman_joint" type="fixed">
+        <parent link="${lr_prefix}_${fr_prefix}_wheel"/>
+        <child link="${lr_prefix}_${fr_prefix}_wheel_axis"/>
+      </joint>
+    </xacro:if>
   </xacro:macro>
   <!-- xacro:macro name="rubber_wheel" params="name parent *origin reflect hq" -->
@@ -216,6 +232,6 @@
       <type>transmission_interface/SimpleTransmission</type>
       <joint name="${lr_prefix}_steering_joint">
-        <!--<hardwareInterface>hardware_interface/EffortJointInterface</hardwareInterface>-->
-        <hardwareInterface>hardware_interface/PositionJointInterface</hardwareInterface>
+        <hardwareInterface>hardware_interface/EffortJointInterface</hardwareInterface>
+        <!-- <hardwareInterface>hardware_interface/PositionJointInterface</hardwareInterface> -->
       </joint>
       <actuator name="${lr_prefix}_steering_act">

Commit message: Added HQ model and changed control for more stable system in noetic

File: rbcar_description/robots/versions/rbcar_roborder.urdf.xacro (robot description, xacro)
@@ -9,5 +9,7 @@
 	<xacro:include filename="$(find rbcar_description)/urdf/bases/rbcar_base.urdf.xacro" />
 	<!-- Import Robotnik CAR wheels -->
-	<xacro:include filename="$(find rbcar_description)/urdf/wheels/suspension_wheel_v3.urdf.xacro" />
+	<!-- <xacro:include filename="$(find rbcar_description)/urdf/wheels/suspension_wheel_v3.urdf.xacro" /> -->
+  <xacro:include filename="$(find rbcar_description)/urdf/common/macros.xacro" />
+  <xacro:include filename="$(find rbcar_description)/urdf/wheels/wheels.xacro" />
 	<xacro:include filename="$(find rbcar_description)/urdf/structures/elevator.urdf.xacro" />
 	<!-- Import all available sensors -->
@@ -26,9 +28,10 @@
 	<!-- Flag to select the high or low quality model -->
 	<xacro:property name="hq" value="true" />
+  <!-- Argument for Setting the Wheel Ackerman visual help Is set as argument in the Wheels.xacro, so take that into account-->
 	<!-- *************** -->
 	<!-- Robots Elements -->
 	<!-- *************** -->
 	<!-- Here we create the robot elements using the xacro:macros imported at the beggining of this file -->
-	<!-- Summit XL base -->
+	<!-- RB CAR BASE -->
 	<xacro:rbcar_base name="roborder" publish_bf="true" hq="${hq}" />
 	<!-- Gazebo ros control pluggins -->
@@ -39,5 +42,5 @@
 	<!-- WHEELS -->
   <!-- Wheels -->
-  <xacro:front_wheel lr_prefix="left" fr_prefix="front"
+  <!-- <xacro:front_wheel lr_prefix="left" fr_prefix="front"
                      lr_reflect="1" fr_reflect="1" parent="base_link" />
   <xacro:front_wheel lr_prefix="right" fr_prefix="front"
@@ -46,7 +49,7 @@
                     lr_reflect="1" fr_reflect="-1" parent="base_link" />
   <xacro:rear_wheel lr_prefix="right" fr_prefix="rear"
-                    lr_reflect="-1" fr_reflect="-1" parent="base_link" />
+                    lr_reflect="-1" fr_reflect="-1" parent="base_link" />    -->
 	<!-- SENSORS -->
-  <xacro:elevator parent="base_link">
+  <xacro:elevator parent="base_link" fixed_elevator="false">
 		<origin xyz="0.0 0.0 0.6" rpy="0 0 0"/>
 	</xacro:elevator>
@@ -55,7 +58,8 @@
 	</xacro:sensor_imu_hector>
 	<xacro:sensor_gps prefix="gps" parent="base_link" gps_latitude="$(arg gps_latitude)" gps_longitude="$(arg gps_longitude)" update_rate="20" >
-		<origin xyz="0.0 0 1.5" rpy="0 0 0"/>
+		<origin xyz="0.0 0 0.0" rpy="0 0 0"/>
 	</xacro:sensor_gps>
-  <xacro:sensor_benewake_ce30d prefix="front_ss_lidar" parent="base_link" prefix_topic='front_ss_lidar' gpu="false">
+  <!-- The Solid State Lydars in Four directions Front , Rear, Left and Right-->
+  <!-- <xacro:sensor_benewake_ce30d prefix="front_ss_lidar" parent="base_link" prefix_topic='front_ss_lidar' gpu="false">
       <origin xyz="2.155 0.0 0.236" rpy="0 0 0"/>
   </xacro:sensor_benewake_ce30d>
@@ -64,16 +68,22 @@
   </xacro:sensor_benewake_ce30d>
   <xacro:sensor_benewake_ce30d prefix="left_ss_lidar" parent="base_link" prefix_topic='left_ss_lidar' gpu="false">
-      <origin xyz="1.0 -0.8 0.236" rpy="0 0 -1.52"/>
+      <origin xyz="1.0 -0.7 0.236" rpy="0 0 -1.52"/>
   </xacro:sensor_benewake_ce30d>
   <xacro:sensor_benewake_ce30d prefix="right_ss_lidar" parent="base_link" prefix_topic='right_ss_lidar' gpu="false">
-      <origin xyz="1.0 0.8 0.236" rpy="0 0 1.52"/>
-  </xacro:sensor_benewake_ce30d>
-  <xacro:sensor_axis_q8641 prefix="front_ptz_camera" parent="elevator_link" far="300" near="0.08">
-    <origin xyz="0 0 0" rpy="0 0 0"/>
-  </xacro:sensor_axis_q8641>
+      <origin xyz="1.0 0.7 0.236" rpy="0 0 1.52"/>
+  </xacro:sensor_benewake_ce30d> -->
+  <!-- <xacro:sensor_axis_q8641 prefix="front_ptz_camera" parent="base_link" far="300" near="0.08">
+    <origin xyz="0 0 2.0" rpy="0 0 0"/>
+  </xacro:sensor_axis_q8641> -->
+  <xacro:sensor_hokuyo_utm30lx prefix="hokuyo_front_laser" parent="base_link" prefix_topic='hokuyo_front_laser' gpu="false" min_angle="-1.57" max_angle="1.57">
+      <origin xyz="2.22193 0.0 0.055082" rpy="0 0 0"/>
+  </xacro:sensor_hokuyo_utm30lx>
   <!-- Adding Sensors for navigation - and autonomous driving . Custom vvalues due to instability of version 16-->
-  <!-- <xacro:sensor_rslidar prefix="rslidar" parent="elevator_link" prefix_topic="rslidar" range_min="0.2" range_max="150.0" hfov="360.0" hres="0.1" vfov="30.0" vres="0.2" fps="2.0" gpu="true">
+  <!-- <xacro:sensor_rslidar prefix="rslidar" parent="elevator_link" prefix_topic="rslidar" range_min="0.2" range_max="50.0" hfov="360.0" hres="0.4" vfov="30.0" vres="0.8" fps="2.0" gpu="true">
     <origin xyz="0 0 0" rpy="0 0 0"/>
   </xacro:sensor_rslidar> -->
+  <xacro:sensor_mpc3_bosch prefix="ueye_rgb_camera" parent="base_link">
+      <origin xyz="1.32236 0.013835 1.48042" rpy="0 0 0"/>
+  </xacro:sensor_mpc3_bosch>
 <gazebo>
 <plugin name="ground_truth_controller" filename="librobotnik_gazebo_ground_truth_odom.so">

File: rbcar_description/urdf/bases/rbcar_base.urdf.xacro (robot description, xacro)
@@ -7,4 +7,5 @@
   <xacro:property name="wheel_width" value="0.317" />
   <xacro:property name="clearance" value="${tire_dia/2.0}" />
+  <xacro:property name="chassis_mass" value="125.0" />
   <!-- BASE FOOTPRINT -->
   <xacro:if value="${publish_bf}">
@@ -34,7 +35,8 @@
   <link name="${prefix}base_link">
     <inertial>
-      <mass value="125.0" />
+      <mass value="${chassis_mass}" />
       <origin xyz="0.917 0 0" />
-      <inertia  ixx="1.391" ixy="0.004"  ixz="0.0"  iyy="6.853"  iyz="0.0"  izz="6.125" />
+      <xacro:box_inertia mass="${chassis_mass}" x="2.59697" y="1.38479" z="1.65615"/>
+      <!-- <inertia  ixx="1.391" ixy="0.004"  ixz="0.0"  iyy="6.853"  iyz="0.0"  izz="6.125" /> -->
     </inertial>
     <visual>
@@ -42,5 +44,5 @@
        <xacro:if value="${hq}">
        <geometry>
-	     <mesh filename="package://rbcar_description/meshes/bases/rbcar_chassis_hq.stl"/>
+	     <mesh filename="package://rbcar_description/meshes/bases/rbcar_hq.dae" scale="1.0 1.0 1.0"/>
        </geometry>
        </xacro:if>

File: rbcar_description/urdf/structures/elevator.urdf.xacro (robot description, xacro)
@@ -8,5 +8,5 @@
   <xacro:property name="outer_radius" value="0.07" />
   <xacro:property name="inner_radius" value="0.05" />
-  <xacro:macro name="elevator" params="prefix:='' parent *origin">
+  <xacro:macro name="elevator" params="prefix:='' parent *origin fixed_elevator:=true">
     <xacro:macro name="solid_cuboid_inertia" params="m h d w">
       <inertia ixx="${(m*(h*h+d*d))/12}" ixy = "0" ixz = "0" iyy="${(m*(w*w+d*d))/12}" iyz = "0" izz="${(m*(w*w+h*h))/12}" />
@@ -25,4 +25,10 @@
         </geometry>
       </visual>
+      <collision>
+        <origin xyz="0 0 ${length/2.0}" rpy="0 0 0" />
+        <geometry>
+            <cylinder radius="${outer_radius}" length="${length}"/>
+        </geometry>
+      </collision>
       <inertial>
         <mass value="1" />
@@ -31,13 +37,4 @@
       </inertial>
     </link>
-    <!-- Elevator structure -->
-    <joint name="${prefix}elevator_joint" type="prismatic">
-      <parent link="${prefix}elevator_base_link"/>
-      <origin xyz="0.0 0.0 ${length}" rpy="0 0 0" />
-      <child link="${prefix}elevator_link"/>
-      <axis xyz="0 0 1"/>
-      <limit lower="0.0" upper="${spread}" effort="1000.0" velocity="0.07"/>
-      <!--<xacro:insert_block name="origin" />-->
-    </joint>
     <link name="${prefix}elevator_link">
       <visual>
@@ -47,4 +44,10 @@
         </geometry>
       </visual>
+      <collision>
+        <origin xyz="0 0 -${length/2.0}" rpy="0 0 0" />
+        <geometry>
+            <cylinder radius="${inner_radius}" length="${length}"/>
+        </geometry>
+      </collision>
       <inertial>
         <mass value="0.1" />
@@ -53,16 +56,32 @@
       </inertial>
     </link>
-    <transmission name="${prefix}elevator_trans">
+    <!-- Elevator structure Fixed by default because unstable due to Gazebo Physiscs-->
+    <xacro:if value="${fixed_elevator}">
+      <joint name="${prefix}elevator_joint" type="fixed">
+        <parent link="${prefix}elevator_base_link"/>
+        <origin xyz="0.0 0.0 ${length + 0.3}" rpy="0 0 0" />
+        <child link="${prefix}elevator_link"/>
+      </joint>
+    </xacro:if>
+    <xacro:unless value="${fixed_elevator}">
+      <joint name="${prefix}elevator_joint" type="prismatic">
+        <parent link="${prefix}elevator_base_link"/>
+        <origin xyz="0.0 0.0 ${length}" rpy="0 0 0" />
+        <child link="${prefix}elevator_link"/>
+        <axis xyz="0 0 1"/>
+        <limit lower="0.3" upper="${spread}" effort="10000.0" velocity="0.01"/>
+        <joint_properties damping="1.0" friction="10.0"/>
+      </joint>
+      <transmission name="${prefix}elevator_trans">
       <type>transmission_interface/SimpleTransmission</type>
       <joint name="${prefix}elevator_joint">
         <hardwareInterface>hardware_interface/EffortJointInterface</hardwareInterface>
-        <!-- <hardwareInterface>hardware_interface/PositionJointInterface</hardwareInterface> -->
       </joint>
       <actuator name="${prefix}elevator_motor">
         <mechanicalReduction>1</mechanicalReduction>
         <hardwareInterface>hardware_interface/EffortJointInterface</hardwareInterface>
-        <!-- <hardwareInterface>hardware_interface/PositionJointInterface</hardwareInterface> -->
       </actuator>
     </transmission>
+    </xacro:unless>
   </xacro:macro>
 </robot>

File: rbcar_description/urdf/wheels/suspension_wheel_v3.urdf.xacro (robot description, xacro)
@@ -69,5 +69,5 @@
     <inertial>
       <mass value="0.001"/>
-      <inertia ixx="0.001" ixy="0" ixz="0" iyy="0.001" iyz="0" izz="0.001"/>
+      <inertia ixx="1.6666666666666666e-10" ixy="0" ixz="0" iyy="1.6666666666666666e-10" iyz="0" izz="1.6666666666666666e-10"/>
     </inertial>
   </xacro:macro>
